File: kicad/nrg-control-box.kicad_pcb (KiCad board)
At the start: 2 copper layers, 35.5 x 33.5 mm, 35 parts, among them J1 OLED, J2 NRG, J3 AVR-ISP-6, J4 USB, SW1 RESET, U1 LM321, U2 SN74LVC1G14DBV, U3 ATmega32U4-AU, U4 XC6210, Y1 8MHz

Commit message: updated schematic to reflect change in measurement pin to PC7
Connections:
- U3 pad 32: Net-(U3-Pad32) -> Net-(R5-Pad1)
Routing:
- net Net-(R5-Pad1): track 20.3 -> 27.7 mm, vias 1 -> 2
