File: kicad/nrg-control-box.sch (KiCad schematic (older format))
At the start: 30 parts, among them J1 OLED, J2 NRG, J3 AVR-ISP-6, J4 USB, SW1 RESET, U1 LM321, U3 ATmega32U4-AU, U4 XC6210, Y1 8MHz

Commit message: updated schematic to reflect change in measurement pin to PC7
Parts:
- J4: symbol Connector:USB_B_Micro -> nrg-control-box-rescue:USB_B_Micro-Connector
Connections:
- net at R5.1, TP2.1, U1.4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: now also U3.32 (PC7)
- no-connect marks 22 -> 21
Changed lines of the file:
@@
 Sheet 1 1
 Title "NRG Anemometer Display"
-Date "2020-09-14"
-Rev "B"
+Date "2021-02-07"
+Rev "C"
 Comp "W3AXL"
 Comment1 ""
@@
 	3400 5150 3400 5200
 $Comp
-L Connector:USB_B_Micro J4
+L nrg-control-box-rescue:USB_B_Micro-Connector J4
 U 1 1 5F46D984
 P 9200 3250
@@
 Connection ~ 7650 1950
 NoConn ~ 6350 3150
-NoConn ~ 6350 3250
 NoConn ~ 6350 4750
 NoConn ~ 6350 4850
@@
 NoConn ~ 6350 4450
 Wire Wire Line
-	4300 4650 6350 4650
+	4300 4650 5500 4650
 Connection ~ 4300 4650
+Wire Wire Line
+	6350 3250 5500 3250
+Wire Wire Line
+	5500 3250 5500 4650
+Connection ~ 5500 4650
+Wire Wire Line
+	5500 4650 6350 4650
 $EndSCHEMATC
